File: WLR089U0-DevBoard.sch (KiCad schematic (older format))
At the start: 26 parts, among them IC1 WLR089U0-I_RM, J1 USB_B_Micro, J10 Conn_01x04_Male, J2 Conn_01x08_Female, J3 Conn_ARM_JTAG_SWD_10, J4 Conn_01x05_Female, J5 Conn_01x08_Female, J6 Conn_01x04_Male, J8 Conn_01x06_Male, J9 Conn_01x06_Male, U1 MCP1700-3302E_SOT23, U2 CH340G

Commit message: edited schematic
Parts:
- removed C3: 100n, symbol Device:C_Small
- IC1: symbol SamacSys_Parts:WLR089U0-I_RM -> WLR089U0-DevBoard-rescue:WLR089U0-I_RM-SamacSys_Parts
- J1: symbol Connector:USB_B_Micro -> WLR089U0-DevBoard-rescue:USB_B_Micro-Connector
Connections:
- net labels added: +3V3
- wire segments 72 -> 73
Changed lines of the file:
@@
 EESchema Schematic File Version 4
-LIBS:LoRa wan-cache
 EELAYER 30 0
 EELAYER END
@@
 $EndDescr
 $Comp
-L SamacSys_Parts:WLR089U0-I_RM IC1
+L WLR089U0-DevBoard-rescue:WLR089U0-I_RM-SamacSys_Parts IC1
 U 1 1 601A9C3D
 P 2100 2550
@@
 	2400 1150 2400 1450
 $Comp
-L Connector:USB_B_Micro J1
+L WLR089U0-DevBoard-rescue:USB_B_Micro-Connector J1
 U 1 1 601E6237
 P 950 1350
@@
 Wire Wire Line
 	5000 850  5000 1050
-Text GLabel 4100 1150 2    50   Input ~ 0
-+3V
 NoConn ~ 2100 6200
 Text GLabel 6000 2900 2    50   Input ~ 0
@@
 Wire Wire Line
 	3800 1150 4100 1150
-Text GLabel 4700 850  1    50   Input ~ 0
-+3V
 Wire Wire Line
 	4700 850  4700 1100
@@
 	1    0    0    -1
 $EndComp
-Text GLabel 4400 2500 1    50   Input ~ 0
-+3V
 $Comp
 L Device:R_Small R6
@@
 Wire Wire Line
 	4400 2500 4400 2600
-$Comp
-L Device:C_Small C3
-U 1 1 602CE99D
-P 4400 3000
-F 0 "C3" H 4492 3046 50  0000 L CNN
-F 1 "100n" H 4492 2955 50  0000 L CNN
-F 2 "" H 4400 3000 50  0001 C CNN
-F 3 "~" H 4400 3000 50  0001 C CNN
-	1    4400 3000
-	1    0    0    -1
-$EndComp
 Text GLabel 3500 2850 2    50   Input ~ 0
 RESET
@@
 L power:GND #PWR?
 U 1 1 602CF171
-P 4400 3250
-F 0 "#PWR?" H 4400 3000 50  0001 C CNN
-F 1 "GND" H 4405 3077 50  0000 C CNN
-F 2 "" H 4400 3250 50  0001 C CNN
-F 3 "" H 4400 3250 50  0001 C CNN
-	1    4400 3250
+P 4400 3380
+F 0 "#PWR?" H 4400 3130 50  0001 C CNN
+F 1 "GND" H 4405 3207 50  0000 C CNN
+F 2 "" H 4400 3380 50  0001 C CNN
+F 3 "" H 4400 3380 50  0001 C CNN
+	1    4400 3380
 	1    0    0    -1
 $EndComp
@@
 	4400 2800 4400 2850
 Wire Wire Line
-	4400 3100 4400 3250
+	4400 3230 4400 3380
 Wire Wire Line
 	4400 2850 4600 2850
@@
 	1    0    0    -1
 $EndComp
+$Comp
+L power:+3V3 #PWR?
+U 1 1 601BD609
+P 4100 1120
+F 0 "#PWR?" H 4100 970 50  0001 C CNN
+F 1 "+3V3" H 4115 1293 50  0000 C CNN
+F 2 "" H 4100 1120 50  0001 C CNN
+F 3 "" H 4100 1120 50  0001 C CNN
+	1    4100 1120
+	1    0    0    -1
+$EndComp
+Wire Wire Line
+	4100 1120 4100 1150
+$Comp
+L power:+3V3 #PWR?
+U 1 1 601C0F1A
+P 4700 850
+F 0 "#PWR?" H 4700 700 50  0001 C CNN
+F 1 "+3V3" H 4715 1023 50  0000 C CNN
+F 2 "" H 4700 850 50  0001 C CNN
+F 3 "" H 4700 850 50  0001 C CNN
+	1    4700 850
+	1    0    0    -1
+$EndComp
+$Comp
+L power:+3V3 #PWR?
+U 1 1 601C1722
+P 4400 2500
+F 0 "#PWR?" H 4400 2350 50  0001 C CNN
+F 1 "+3V3" H 4415 2673 50  0000 C CNN
+F 2 "" H 4400 2500 50  0001 C CNN
+F 3 "" H 4400 2500 50  0001 C CNN
+	1    4400 2500
+	1    0    0    -1
+$EndComp

Commit message: Edited power symbols, ch340e needs to be made
Parts:
- removed J10: Conn_01x04_Male, symbol Connector:Conn_01x04_Male
- removed J9: Conn_01x06_Male, symbol Connector:Conn_01x06_Male
Connections:
- wire segments 73 -> 63
Other:
- moved on the sheet: C1, C2, C4, D1, J1, J3, JP1, JP2, R1, U1

Commit message: Power supply done and ch304e remaining
Parts:
- added SW1: SW_Push, symbol Switch:SW_Push
- gave numbers to parts that had none: 1
- renumbered R6 to R2
Connections:
- net labels removed: +3V
- wire segments 63 -> 104
Other:
- moved on the sheet: R2

Commit message: pins changed and ch304e symbol done
Parts:
- removed J2, J5: Conn_01x08_Female, symbol Connector:Conn_01x08_Female
- removed J4: Conn_01x05_Female, symbol Connector:Conn_01x05_Female
- removed U2: CH340G, Package_SO:SOIC-16_3.9x9.9mm_P1.27mm, symbol Interface_USB:CH340G
- added J2, J3: Conn_01x10_Female, symbol Connector:Conn_01x10_Female
- added U4: CH304e, symbol Interface_USB:CH304e
Connections:
- wire segments 104 -> 102
- no-connect marks 11 -> 5
Other:
- moved on the sheet: D2, IC1, JP1, JP2, R2, R3, SW1

Commit message: pins done and symbol ch304e
Connections:
- wire segments 102 -> 110
Other:
- moved on the sheet: J3, JP1
Changed lines of the file:
@@
 Text GLabel 1400 3500 0    50   Input ~ 0
 PA08
-Text GLabel 6500 3950 2    50   Input ~ 0
+Text GLabel 6550 3240 0    50   Input ~ 0
 PA27
 Text GLabel 1400 3800 0    50   Input ~ 0
@@
 Text GLabel 1400 3600 0    50   Input ~ 0
 PA14
-Text GLabel 6500 4050 2    50   Input ~ 0
+Text GLabel 6550 3140 0    50   Input ~ 0
 PA22
 Text GLabel 3100 3100 0    50   Input ~ 0
@@
 Text GLabel 1400 3200 0    50   Input ~ 0
 PA03
-Text GLabel 6500 3850 2    50   Input ~ 0
+Text GLabel 6550 3340 0    50   Input ~ 0
 PA28
-Text GLabel 6550 3650 2    50   Input ~ 0
+Text GLabel 6500 3540 0    50   Input ~ 0
 VDDCORE
-Text GLabel 6550 3750 2    50   Input ~ 0
+Text GLabel 6500 3440 0    50   Input ~ 0
 VSW
 Text GLabel 4500 2700 2    50   Input ~ 0
@@
 Wire Wire Line
 	1060 1260 1360 1260
-Text GLabel 3815 6505 3    50   Input ~ 0
+Text GLabel 3860 6500 3    50   Input ~ 0
 D+
 Text GLabel 3615 7205 3    50   Input ~ 0
@@
 L Jumper:SolderJumper_3_Bridged12 JP1
 U 1 1 602772DE
-P 3815 6205
-F 0 "JP1" H 3665 6055 50  0000 C CNN
-F 1 "SolderJumper_3_Bridged12" H 3815 6319 50  0000 C CNN
-F 2 "" H 3815 6205 50  0001 C CNN
-F 3 "~" H 3815 6205 50  0001 C CNN
-	1    3815 6205
+P 3860 6200
+F 0 "JP1" H 3710 6050 50  0000 C CNN
+F 1 "SolderJumper_3_Bridged12" H 3860 6314 50  0000 C CNN
+F 2 "" H 3860 6200 50  0001 C CNN
+F 3 "~" H 3860 6200 50  0001 C CNN
+	1    3860 6200
 	-1   0    0    -1
 $EndComp
@@
 	3615 7005 3615 7205
 Wire Wire Line
-	3815 6355 3815 6505
-Text GLabel 3415 6205 0    50   Input ~ 0
+	3860 6350 3860 6500
+Text GLabel 3460 6200 0    50   Input ~ 0
 MCU_U_P
 Text GLabel 3265 6855 0    50   Input ~ 0
@@
 	3265 6855 3415 6855
 Wire Wire Line
-	3415 6205 3615 6205
+	3460 6200 3660 6200
 $Comp
 L Jumper:SolderJumper_2_Bridged JP3
@@
 L power:+3V3 #PWR?
 U 1 1 601BD6AD
-P 6550 3350
-F 0 "#PWR?" H 6550 3200 50  0001 C CNN
-F 1 "+3V3" H 6565 3523 50  0000 C CNN
-F 2 "" H 6550 3350 50  0001 C CNN
-F 3 "" H 6550 3350 50  0001 C CNN
-	1    6550 3350
-	0    1    1    0
+P 6500 3840
+F 0 "#PWR?" H 6500 3690 50  0001 C CNN
+F 1 "+3V3" H 6515 4013 50  0000 C CNN
+F 2 "" H 6500 3840 50  0001 C CNN
+F 3 "" H 6500 3840 50  0001 C CNN
+	1    6500 3840
+	0    -1   -1   0
 $EndComp
 $Comp
@@
 	0    1    1    0
 $EndComp
-Text GLabel 6550 3550 2    50   Input ~ 0
+Text GLabel 6500 3640 0    50   Input ~ 0
 UART_RX
-Text GLabel 6550 3450 2    50   Input ~ 0
+Text GLabel 6500 3740 0    50   Input ~ 0
 UART_TX
 $Comp
@@
 	1    0    0    -1
 $EndComp
-$Comp
-L Connector:Conn_01x10_Female J3
-U 1 1 601E7A94
-P 6150 3650
-F 0 "J3" V 6223 3580 50  0000 C CNN
-F 1 "Conn_01x10_Female" V 6314 3580 50  0000 C CNN
-F 2 "" H 6150 3650 50  0001 C CNN
-F 3 "~" H 6150 3650 50  0001 C CNN
-	1    6150 3650
-	-1   0    0    1
-$EndComp
 Wire Wire Line
 	1100 4000 1400 4000
@@
 	1100 4100 1400 4100
 Wire Wire Line
-	6350 4050 6500 4050
-Wire Wire Line
-	6350 3950 6500 3950
-Wire Wire Line
-	6350 3850 6500 3850
-Wire Wire Line
-	6350 3750 6550 3750
-Wire Wire Line
-	6350 3650 6550 3650
-Wire Wire Line
-	6350 3550 6550 3550
-Wire Wire Line
-	6350 3450 6550 3450
-Wire Wire Line
-	6350 3350 6550 3350
+	6700 3140 6550 3140
+Wire Wire Line
+	6700 3240 6550 3240
+Wire Wire Line
+	6700 3440 6500 3440
+Wire Wire Line
+	6700 3540 6500 3540
+Wire Wire Line
+	6700 3640 6500 3640
+Wire Wire Line
+	6700 3740 6500 3740
+Wire Wire Line
+	6700 3840 6500 3840
 $Comp
 L power:GND #PWR?
 U 1 1 60245A07
-P 6550 3100
-F 0 "#PWR?" H 6550 2850 50  0001 C CNN
-F 1 "GND" H 6555 2927 50  0000 C CNN
-F 2 "" H 6550 3100 50  0001 C CNN
-F 3 "" H 6550 3100 50  0001 C CNN
-	1    6550 3100
-	0    -1   -1   0
-$EndComp
-Wire Wire Line
-	6350 3250 6550 3250
-Wire Wire Line
-	6550 3250 6550 3150
-Wire Wire Line
-	6350 3150 6550 3150
-Connection ~ 6550 3150
-Wire Wire Line
-	6550 3150 6550 3100
+P 6500 4090
+F 0 "#PWR?" H 6500 3840 50  0001 C CNN
+F 1 "GND" H 6505 3917 50  0000 C CNN
+F 2 "" H 6500 4090 50  0001 C CNN
+F 3 "" H 6500 4090 50  0001 C CNN
+	1    6500 4090
+	0    1    1    0
+$EndComp
+Wire Wire Line
+	6700 3940 6500 3940
+Wire Wire Line
+	6500 3940 6500 4040
+Wire Wire Line
+	6700 4040 6500 4040
+Connection ~ 6500 4040
+Wire Wire Line
+	6500 4040 6500 4090
 Wire Wire Line
 	5400 3400 5400 3150
@@
 $EndComp
 Wire Wire Line
-	4715 5755 5365 5755
+	4715 5755 4800 5755
 $Comp
 L Interface_USB:CH304e U4
@@
 	4950 7200 4950 7350
 Wire Wire Line
-	4000 6200 4500 6200
-Wire Wire Line
 	4500 6350 4150 6350
-Wire Wire Line
-	4150 6350 4150 6850
-Wire Wire Line
-	4150 6850 3800 6850
-Wire Wire Line
-	4800 5750 4800 5900
-Wire Wire Line
-	4950 5750 4950 5900
 NoConn ~ 5350 6650
 NoConn ~ 5350 6900
 NoConn ~ 4500 6650
+Wire Wire Line
+	5390 6155 5765 6155
+Wire Wire Line
+	5350 6200 5390 6200
+Wire Wire Line
+	5390 6155 5390 6200
+Wire Wire Line
+	5605 6350 5605 6255
+Wire Wire Line
+	5605 6255 5765 6255
+Wire Wire Line
+	5350 6350 5605 6350
+Wire Wire Line
+	3815 6855 4150 6855
+Wire Wire Line
+	4150 6350 4150 6855
+Wire Wire Line
+	4060 6200 4500 6200
+Wire Wire Line
+	4800 5900 4800 5755
+Connection ~ 4800 5755
+Wire Wire Line
+	4800 5755 4950 5755
+Wire Wire Line
+	4950 5900 4950 5755
+Connection ~ 4950 5755
+Wire Wire Line
+	4950 5755 5365 5755
+Wire Wire Line
+	6700 3340 6550 3340
+$Comp
+L Connector:Conn_01x10_Female J3
+U 1 1 601E7A94
+P 6900 3540
+F 0 "J3" V 6973 3470 50  0000 C CNN
+F 1 "Conn_01x10_Female" V 7064 3470 50  0000 C CNN
+F 2 "" H 6900 3540 50  0001 C CNN
+F 3 "~" H 6900 3540 50  0001 C CNN
+	1    6900 3540
+	1    0    0    -1
+$EndComp
 $EndSCHEMATC

Commit message: blue box and final version done
Connections:
- wire segments 110 -> 109
Other:
- note added: "POWER CURCUITRY"
- note added: "Programming unit"
- note added: "WLR089U0-SAMR34-Dev-Board-LoRaWAN"
- moved on the sheet: C1, C2, C4, D1, D2, IC1, J1, J2, J3, JP1, JP2, R1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

Commit message: Beautified schematic layout, ERC pending
Parts:
- removed J6: Conn_01x04_Male, symbol Connector:Conn_01x04_Male
- removed JP3, JP4, JP5: SolderJumper_2_Bridged, symbol Jumper:SolderJumper_2_Bridged
- removed U4: CH304e, symbol Interface_USB:CH304e
- added JP3: SolderJumper_2_Open, symbol Jumper:SolderJumper_2_Open
- added U2: CH304E, symbol WLR089U0-DevBoard-rescue:CH304E
- J4: renamed from J8; value Conn_01x06_Male -> Conn_01x10_Male; symbol Connector:Conn_01x06_Male -> Connector:Conn_01x10_Male
- renumbered C4 to C3, J3 to J2, J2 to J3, J3 to J5, JP2 to JP1, JP1 to JP2, R2 to R1, R1 to R2
Connections:
- net labels removed: SWCLK
- wire segments 109 -> 114
Other:
- note added: "ARM CORTEX SWD PROGRAMMING\n10 PIN HEADER"
- note added: "BLANK SPACE"
- note added: "GPIO PIN HEADERS"
- note added: "GPIO STATUS LED"
- note added: "I2C & SPI HEADER"
- note added: "Microchip WLR089U0-SAMR34 Module"
- note added: "POWER CIRCUITRY"
- note added: "POWER LED"
- note added: "USB-UART USING CH340E via JP3 short (OR)\nUSB-USB via JP1,JP2 short"
- note removed: "POWER CURCUITRY"
- note removed: "Programming unit"
- note removed: "WLR089U0-SAMR34-Dev-Board-LoRaWAN"
- moved on the sheet: C1, C2, C3, D1, D2, IC1, J1, J2, J3, J5, JP1, JP2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

Commit message: final schematic
Parts:
- D2: value orange -> Green
Connections:
- net +3V3: now also JP3.1 (A); no longer JP3.2 (B)
- net at C3.1, U2.10 (V3), U2.7 (VCC): now also JP3.2 (B); no longer JP3.1 (A)
Other:
- moved on the sheet: C3
Changed lines of the file:
@@
 EESchema Schematic File Version 4
+LIBS:WLR089U0-DevBoard-cache
 EELAYER 30 0
 EELAYER END
@@
 P 6350 1265
 F 0 "D2" V 6396 1197 50  0000 R CNN
-F 1 "orange " V 6305 1197 50  0000 R CNN
+F 1 "Green" V 6305 1197 50  0000 R CNN
 F 2 "" V 6350 1265 50  0001 C CNN
 F 3 "~" V 6350 1265 50  0001 C CNN
@@
 L Device:C_Small C3
 U 1 1 602D3CA5
-P 9335 3045
-F 0 "C3" V 9564 3045 50  0000 C CNN
-F 1 "100n" V 9473 3045 50  0000 C CNN
-F 2 "" H 9335 3045 50  0001 C CNN
-F 3 "~" H 9335 3045 50  0001 C CNN
-	1    9335 3045
+P 9125 3045
+F 0 "C3" V 9354 3045 50  0000 C CNN
+F 1 "100n" V 9263 3045 50  0000 C CNN
+F 2 "" H 9125 3045 50  0001 C CNN
+F 3 "~" H 9125 3045 50  0001 C CNN
+	1    9125 3045
 	0    -1   -1   0
 $EndComp
@@
 L power:GND #PWR022
 U 1 1 602D61C1
-P 9635 3045
-F 0 "#PWR022" H 9635 2795 50  0001 C CNN
-F 1 "GND" V 9640 2917 50  0000 R CNN
-F 2 "" H 9635 3045 50  0001 C CNN
-F 3 "" H 9635 3045 50  0001 C CNN
-	1    9635 3045
+P 9425 3045
+F 0 "#PWR022" H 9425 2795 50  0001 C CNN
+F 1 "GND" V 9430 2917 50  0000 R CNN
+F 2 "" H 9425 3045 50  0001 C CNN
+F 3 "" H 9425 3045 50  0001 C CNN
+	1    9425 3045
 	0    -1   -1   0
 $EndComp
 Wire Wire Line
-	9435 3045 9635 3045
+	9225 3045 9425 3045
 $Comp
 L Regulator_Linear:MCP1700-3302E_SOT23 U1
@@
 	1    0    0    -1
 $EndComp
-Wire Wire Line
-	8820 3045 8970 3045
-Connection ~ 8970 3045
 Text Notes 570  5465 0    79   ~ 16
 ARM CORTEX SWD PROGRAMMING\n10 PIN HEADER
@@
 	1650 7260 1600 7260
 Connection ~ 1600 7260
-Wire Wire Line
-	8970 3045 9235 3045
 Text GLabel 9740 3640 2    50   Input ~ 0
 UART_TX
@@
 Wire Wire Line
 	8075 4175 8395 4175
-$Comp
-L Jumper:SolderJumper_2_Open JP3
-U 1 1 6031D154
-P 8570 3045
-F 0 "JP3" H 8570 2875 50  0000 C CNN
-F 1 "SolderJumper_2_Open" H 8565 2945 50  0000 C CNN
-F 2 "" H 8570 3045 50  0001 C CNN
-F 3 "~" H 8570 3045 50  0001 C CNN
-	1    8570 3045
-	-1   0    0    1
-$EndComp
-Wire Wire Line
-	8720 3045 8820 3045
 Connection ~ 8820 3045
 Wire Wire Line
 	8325 2830 8325 3045
-Wire Wire Line
-	8325 3045 8420 3045
 Text Notes 6950 5340 0    79   ~ 16
 I2C & SPI HEADER
@@
 Text GLabel 4255 6190 0    50   Input ~ 0
 PA07
+$Comp
+L Jumper:SolderJumper_2_Open JP3
+U 1 1 601C47FE
+P 8565 3045
+F 0 "JP3" H 8565 3135 50  0000 C CNN
+F 1 "SolderJumper_2_Open" H 8355 2950 50  0000 C CNN
+F 2 "" H 8565 3045 50  0001 C CNN
+F 3 "~" H 8565 3045 50  0001 C CNN
+	1    8565 3045
+	1    0    0    -1
+$EndComp
+Wire Wire Line
+	8715 3045 8820 3045
+Wire Wire Line
+	8325 3045 8415 3045
+Wire Wire Line
+	8820 3045 8970 3045
+Connection ~ 8970 3045
+Wire Wire Line
+	8970 3045 9025 3045
 $EndSCHEMATC
