File: WLR089U0-DevBoard.kicad_pcb (KiCad board)
At the start: 2 copper layers, 32.2 x 43.1 mm, 23 parts, among them IC1 WLR089U0-I_RM, J1 USB_B_Micro, J2 Conn_ARM_JTAG_SWD_10, J3 Conn_01x10_Female, J4 Conn_01x02_Male, J5 Conn_01x10_Female, J6 Conn_01x08_Male, SW1 SW_Push, U1 MCP1700-3302E_SOT23, U2 CH304E

Commit message: pcb layer remaing
Parts:
- moved C2 9.10 mm to (130.6, 103.2)
- moved C1 7.10 mm to (119.9, 103.0), turned to 0 degrees
- moved U1 4.38 mm to (123.5, 106.4)
- moved J2 4.28 mm to (127.6, 110.3)
- moved J4 4.22 mm to (122.4, 109.5)
- moved C3 4.08 mm to (125.2, 103.2)
- moved J1 3.85 mm to (115.8, 110.5)
- moved JP3 3.83 mm to (109.7, 101.0)
- moved TP1 3.38 mm to (135.3, 109.6)
- moved R2 2.94 mm to (132.9, 106.1), turned to 0 degrees
- moved D1 2.23 mm to (127.7, 106.1), turned to 180 degrees
- moved TP2 2.15 mm to (109.1, 109.8)
- moved U2 1.46 mm to (113.0, 104.1)
- moved JP1 0.96 mm to (108.5, 104.6), turned to 270 degrees
- moved JP2 0.63 mm to (119.1, 105.5), turned to 0 degrees
Other:
- board size 32.2 x 43.1 mm -> 29.9 x 40.1 mm
