File: WLR089U0-DevBoard.kicad_pcb (KiCad board)
At the start: 2 copper layers, 29.9 x 40.1 mm, 23 parts, among them IC1 WLR089U0-I_RM, J1 USB_B_Micro, J2 Conn_ARM_JTAG_SWD_10, J3 Conn_01x10_Female, J4 Conn_01x02_Male, J5 Conn_01x10_Female, J6 Conn_01x08_Male, SW1 SW_Push, U1 MCP1700-3302E_SOT23, U2 CH304E

Commit message: green layer for gnd
Routing:
- added copper zone on B.Cu, net GND
Changed lines of the file:
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@@
   (gr_line (start 137.16 111.4044) (end 137.16 74.8284) (layer Edge.Cuts) (width 0.12))
   (gr_line (start 108.966 113.1316) (end 135.4328 113.1316) (layer Edge.Cuts) (width 0.12))
+  (zone (net 2) (net_name GND) (layer B.Cu) (hatch edge 0.508)
+    (connect_pads (clearance 0.508))
+    (min_thickness 0.254)
+    (fill yes (arc_segments 32) (thermal_gap 0.508) (thermal_bridge_width 0.508))
+    (polygon
+      (pts
+        (xy 106.3244 72.6948) (xy 138.176 72.7964) (xy 138.4808 113.3856) (xy 106.7816 113.3856)
+      )
+    )
+  )
 )

Commit message: routing remaining
Parts:
- moved U2 0.59 mm to (113.6, 104.2)
- moved JP1 0.31 mm to (108.8, 104.6)
Changed lines of the file:
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@@
   )
   (module Jumper:SolderJumper-3_P1.3mm_Bridged12_RoundedPad1.0x1.5mm_NumberLabels (layer F.Cu)
-    (at 108.458 104.5972 270)
+    (at 108.7628 104.6226 270)
     (descr "SMD Solder 3-pad Jumper, 1x1.5mm rounded Pads, 0.3mm gap, pads 1-2 bridged with 1 copper strip, labeled with numbers")
     (tags "solder jumper open")
@@
   )
   (module Package_SO:MSOP-10_3x3mm_P0.5mm (layer F.Cu)
-    (at 112.9792 104.0892 180)
+    (at 113.5634 104.1654 180)
     (descr "10-Lead Plastic Micro Small Outline Package (MS) [MSOP] (see Microchip Packaging Specification 00000049BS.pdf)")
     (tags "SSOP 0.5")
@@
   (gr_arc (start 135.4328 111.4044) (end 135.4328 113.1316) (angle -90) (layer Edge.Cuts) (width 0.12))
   (dimension 40.081232 (width 0.15) (layer Dwgs.User)
-    (gr_text "40.081 mm" (at 139.653798 93.087871 270.0726182) (layer Dwgs.User)
-      (effects (font (size 1 1) (thickness 0.15)))
-    )
-    (feature1 (pts (xy 137.2108 113.1316) (xy 138.965619 113.129376)))
-    (feature2 (pts (xy 137.16 73.0504) (xy 138.914819 73.048176)))
-    (crossbar (pts (xy 138.328399 73.048919) (xy 138.379199 113.130119)))
-    (arrow1a (pts (xy 138.379199 113.130119) (xy 137.791351 112.004359)))
-    (arrow1b (pts (xy 138.379199 113.130119) (xy 138.964192 112.002873)))
-    (arrow2a (pts (xy 138.328399 73.048919) (xy 137.743406 74.176165)))
-    (arrow2b (pts (xy 138.328399 73.048919) (xy 138.916247 74.174679)))
+    (gr_text 40mm (at 139.653797 93.087871 270.1) (layer Dwgs.User)
+      (effects (font (size 1 1) (thickness 0.15)))
+    )
+    (feature1 (pts (xy 137.2108 113.1316) (xy 138.965618 113.129376)))
+    (feature2 (pts (xy 137.16 73.0504) (xy 138.914818 73.048176)))
+    (crossbar (pts (xy 138.328398 73.048919) (xy 138.379198 113.130119)))
+    (arrow1a (pts (xy 138.379198 113.130119) (xy 137.79135 112.004359)))
+    (arrow1b (pts (xy 138.379198 113.130119) (xy 138.964191 112.002873)))
+    (arrow2a (pts (xy 138.328398 73.048919) (xy 137.743405 74.176165)))
+    (arrow2b (pts (xy 138.328398 73.048919) (xy 138.916246 74.174679)))
   )
   (dimension 29.972 (width 0.15) (layer Dwgs.User)
-    (gr_text "29.972 mm" (at 122.2248 115.6816) (layer Dwgs.User)
-      (effects (font (size 1 1) (thickness 0.15)))
-    )
+    (gr_text "30 mm" (at 122.2248 115.6816) (layer Dwgs.User)
+      (effects (font (size 1 1) (thickness 0.15)))
+    )

Commit message: routing done
Routing:
- net +3V3: track 0.00 -> 90.4 mm
- net +5V: track 0.00 -> 58.1 mm, vias 0 -> 2
- net RESET: track 0.00 -> 50.9 mm
- net GND: track 0.00 -> 47.5 mm, vias 0 -> 13
- net S0_UART_TX: track 0.00 -> 40.7 mm, vias 0 -> 1
- net S0_UART_RX: track 0.00 -> 34.6 mm
- net USB_DP: track 0.00 -> 27.1 mm, vias 0 -> 2
- net SWDCLK: track 0.00 -> 25.0 mm, vias 0 -> 1
- net Net-(C3-Pad1): track 0.00 -> 24.3 mm, vias 0 -> 2
- net SWDIO: track 0.00 -> 23.4 mm, vias 0 -> 1
- net PA08: track 0.00 -> 16.3 mm
- net USB_DM: track 0.00 -> 13.5 mm, vias 0 -> 2
- net D+: track 0.00 -> 13.1 mm
- net /3V3: track 0.00 -> 12.9 mm
- net PA07: track 0.00 -> 9.84 mm
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